File: DualHbridgeDaughterboardDesign.kicad_pcb (KiCad board)
At the start: 2 copper layers, 100 x 53.5 mm, 30 parts, among them J1 Screw_Terminal_01x02, J2 Screw_Terminal_01x02, J3 DaughterBoard, J4 Screw_Terminal_01x02, Q1 AOD4189, Q2 AOD4189, Q3 AOD66406, Q4 AOD66406, Q5 AOD4189, Q6 AOD66406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

Commit message: updated a few things
Parts:
- J1, J2, J4: footprint TerminalBlock:TerminalBlock_Altech_AK300-2_P5.00mm -> TerminalBlock_Phoenix:TerminalBlock_Phoenix_MKDS-1,5-2_1x02_P5.00mm_Horizontal
- moved J1 5.10 mm to (81.2, 96.4), turned to -90 degrees
- moved J4 5.00 mm to (112.2, 79.0), turned to 180 degrees
- moved J2 0.40 mm to (165.8, 101.8)
Connections:
- J1 pad 1: /POWB -> /POWA
- J1 pad 2: /POWA -> /POWB
- J4 pad 1: Vdrive -> GND
- J4 pad 2: GND -> Vdrive
Other:
- board text removed: "GP0"
