File: DualHbridgeDaughterboardDesign.kicad_sch (KiCad schematic)
At the start: 29 parts, among them J1 Screw_Terminal_01x02, J2 Screw_Terminal_01x02, J3 DaughterBoard, J4 Screw_Terminal_01x02, Q1 AOD4189, Q2 AOD4189, Q3 AOD66406, Q4 AOD66406, Q5 AOD4189, Q6 AOD66406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

Commit message: updated a few things
Parts:
- J1, J2, J4: footprint TerminalBlock:TerminalBlock_Altech_AK300-2_P5.00mm -> TerminalBlock_Phoenix:TerminalBlock_Phoenix_MKDS-1,5-2_1x02_P5.00mm_Horizontal
Connections:
- net GND: now also J4.1 (Pin_1); no longer J4.2 (Pin_2)
- net POWA: now also J1.1 (Pin_1); no longer J1.2 (Pin_2)
- net POWB: now also J1.2 (Pin_2); no longer J1.1 (Pin_1)
- net Vdrive: now also J4.2 (Pin_2); no longer J4.1 (Pin_1)
Other:
- moved on the sheet: J1, J2, J4
